File: cpm43.kicad_pcb (KiCad board)
At the start: 2 copper layers, 231.3 x 76.8 mm, 185 parts, among them Q1 Q_NPN_BCE, SW1 SW_PUSH, U1 ATmega32U4, U2 PRTR5V0U2X, X1 Crystal_GND24

Commit message: Changed renders
Routing:
- net LEDGND: track 830.1 -> 836.4 mm
Changed lines of the file:
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@@
     (thickness 1.6)
     (drawings 41)
-    (tracks 2367)
+    (tracks 2369)
     (zones 0)
     (modules 185)
@@
   (segment (start 126.8222 72.009) (end 134.5438 72.009) (width 0.127) (layer B.Cu) (net 125))
   (via (at 116.2939 73.1139) (size 0.6) (drill 0.3) (layers F.Cu B.Cu) (net 125))
+  (segment (start 159.21852 130.83032) (end 154.04552 130.83032) (width 0.127) (layer B.Cu) (net 125))
+  (segment (start 160.34552 130.83032) (end 159.21852 130.83032) (width 0.127) (layer B.Cu) (net 125))
   (via (at 234.061 81.153) (size 0.6) (drill 0.3) (layers F.Cu B.Cu) (net 126))
   (segment (start 235.6125 81.102) (end 234.112 81.102) (width 0.127) (layer B.Cu) (net 126))

Commit message: Silkscreen changed
Other:
- board text added: "Pcb designed by Gtrx in collaboration with croa. Github repo: https://github.com/Gtrx0/cpm43"
- board text removed: "Pcb designed by Gtrx in collaboration with Croa. Github repo: https://github.com/Gtrx0/cpm43"
Changed lines of the file:
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@@
     (effects (font (size 1.5 1.5) (thickness 0.3)) (justify mirror))
   )
-  (gr_text "Pcb designed by Gtrx in collaboration with Croa. Github repo: https://github.com/Gtrx0/cpm43" (at 157.099 97.917) (layer B.SilkS)
+  (gr_text "Pcb designed by Gtrx in collaboration with croa. Github repo: https://github.com/Gtrx0/cpm43" (at 157.099 97.917) (layer B.SilkS)
     (effects (font (size 1.5 1.5) (thickness 0.3)) (justify mirror))
   )

Commit message: Edge cut changed, new renders
Parts:
- moved G*** 38.5 mm to (158.6, 122.4)
Other:
- outline, holes or cut-outs redrawn
