File: cpm43.sch (KiCad schematic (older format))
At the start: 53 parts, among them Q1 Q_NPN_BCE, SW1 SW_PUSH, U1 ATmega32U4, U2 PRTR5V0U2X, X1 Crystal_GND24

Commit message: Changed decoupling cap value
Parts:
- added C1: 0.1uf, symbol device:C_Small
- C4: value 0.1uF -> 4.7uF
Changed lines of the file:
@@
 P 16925 10725
 F 0 "C4" H 16935 10795 50  0000 L CNN
-F 1 "0.1uF" H 16935 10645 50  0000 L CNN
+F 1 "4.7uF" H 16935 10645 50  0000 L CNN
 F 2 "Capacitors_SMD:C_0805_HandSoldering" H 16925 10725 50  0001 C CNN
 F 3 "" H 16925 10725 50  0001 C CNN
@@
 	0    -1   -1   0
 $EndComp
+$Comp
+L device:C_Small C1
+U 1 1 5B68FE84
+P 17700 10925
+F 0 "C1" H 17792 10971 50  0000 L CNN
+F 1 "0.1uf" H 17792 10880 50  0000 L CNN
+F 2 "" H 17700 10925 50  0001 C CNN
+F 3 "~" H 17700 10925 50  0001 C CNN
+	1    17700 10925
+	1    0    0    -1
+$EndComp
+Connection ~ 17700 10825
+Connection ~ 17700 11025
 $EndSCHEMATC

Commit message: Added usb breakout header
Parts:
- added J1: Conn_01x04, Pin_Headers:Pin_Header_Straight_1x04_Pitch2.54mm, symbol conn:Conn_01x04
Connections:
- wire segments 275 -> 284
Changed lines of the file:
@@
 	24025 12550 24575 12550
 Wire Wire Line
-	24575 11650 24025 11650
+	24575 11650 24550 11650
 Wire Wire Line
 	24025 11850 24500 11850
@@
 Connection ~ 24100 11950
 Wire Wire Line
-	24100 11950 25925 11950
+	24100 11950 24800 11950
 Wire Wire Line
 	24025 12250 24150 12250
@@
 Connection ~ 24150 12050
 Wire Wire Line
-	24150 12050 25175 12050
+	24150 12050 24875 12050
 Wire Wire Line
 	24425 12800 24750 12800
@@
 Connection ~ 17700 10825
 Connection ~ 17700 11025
+$Comp
+L conn:Conn_01x04 J1
+U 1 1 5B8E0070
+P 25650 10900
+F 0 "J1" H 25730 10892 50  0000 L CNN
+F 1 "Conn_01x04" H 25730 10801 50  0000 L CNN
+F 2 "Pin_Headers:Pin_Header_Straight_1x04_Pitch2.54mm" H 25650 10900 50  0001 C CNN
+F 3 "~" H 25650 10900 50  0001 C CNN
+	1    25650 10900
+	1    0    0    -1
+$EndComp
+Wire Wire Line
+	24550 11650 24550 11100
+Wire Wire Line
+	24550 11100 25450 11100
+Connection ~ 24550 11650
+Wire Wire Line
+	24550 11650 24025 11650
+$Comp
+L power:GND #PWR0105
+U 1 1 5B8F660B
+P 25450 10800
+F 0 "#PWR0105" H 25450 10550 50  0001 C CNN
+F 1 "GND" V 25455 10672 50  0000 R CNN
+F 2 "" H 25450 10800 50  0001 C CNN
+F 3 "" H 25450 10800 50  0001 C CNN
+	1    25450 10800
+	0    1    1    0
+$EndComp
+Wire Wire Line
+	25450 10900 24800 10900
+Wire Wire Line
+	24800 10900 24800 11950
+Connection ~ 24800 11950
+Wire Wire Line
+	24800 11950 25925 11950
+Wire Wire Line
+	25450 11000 24875 11000
+Wire Wire Line
+	24875 11000 24875 12050
+Connection ~ 24875 12050
+Wire Wire Line
+	24875 12050 25175 12050
 $EndSCHEMATC
